File: hardware/version103/_autosave-tmc2209_devboard.kicad_pcb (KiCad board)
At the start: 2 copper layers, 45 x 45 mm, 21 parts, among them J1 Conn_02x05_Odd_Even, J2 Screw_Terminal_01x04, U1 TMC2209-LA

Commit message: Add files via upload
An edited version of Version103 which measures 45x45mm  This one has been ordered through JLCPCB and successfully tested.
Parts:
- added J3: Conn_01x02_Socket, TestPoint:TestPoint_Keystone_5010-5014_Multipurpose, F.Cu at (69.5, 53.7)
- added J4: Conn_01x05_Socket, Connector_PinHeader_2.54mm:PinHeader_1x05_P2.54mm_Vertical, F.Cu at (69.5, 49.4)
- C4: footprint Capacitor_SMD:CP_Elec_5x5.9 -> Capacitor_SMD:CP_Elec_10x10.5
- R9: value R33k -> R20k
- RV1: value R_Potentiometer -> 20k_Potentiometer; footprint Potentiometer_SMD:Potentiometer_Bourns_3214J_Horizontal -> Potentiometer_SMD:Potentiometer_Bourns_3314G_Vertical
- moved C1 4.31 mm to (82.3, 57.6)
- moved C2 4.30 mm to (81.7, 59.9)
- moved C3 4.23 mm to (81.7, 62.5)
- moved C4 2.73 mm to (90.4, 64.1)
- moved R9 2.37 mm to (74.9, 54.4)
- moved RV1 2.03 mm to (76.1, 59.5)
Connections:
- U1 pad 29: unconnected-(U1-EXP-Pad29) -> GND
Routing:
- net unconnected-(U1-~{PD~{_UART}-Pad14): track 18.1 -> 0.00 mm
- net Net-(J3-Pin_1): track 11.3 -> 25.6 mm
- net MOT_INDEX: track 16.3 -> 25.5 mm, vias 0 -> 1
- net MOT_CLK: track 17.2 -> 26.3 mm, vias 0 -> 1
- net MOT_DIAG: track 15.3 -> 22.6 mm, vias 0 -> 1
- net Vdrive: track 51.9 -> 58.4 mm
- net MOT_MS2: track 14.4 -> 19.8 mm, vias 0 -> 1
- net MOT_MS1: track 13.5 -> 17.2 mm, vias 0 -> 1
- net Net-(R9-Pad2): track 6.74 -> 9.85 mm
- net Net-(D2-A): track 0.00 -> 3.02 mm
- net MOT_STEP: track 37.9 -> 36.5 mm
- net MOT_DIR: track 38.1 -> 37.4 mm
- net unconnected-(U1-EXP-Pad29): vias 9 -> 0
- net GND: vias 27 -> 38
Other:
- board text added: "MS1"
- board text added: "MS2"
- board text added: "clk"
- board text added: "diag"
- board text added: "index"
- board text added: "ref. test point"
